File: lab4/lab4/lab4_Exercise2/lab4_Exercise2.kicad_sch (KiCad schematic)
At the start: 10 parts, among them J1 Conn_01x02_Male, U1 NE555D

Commit message: lab4 commit
Parts:
- C1: renamed from C2; value C_Polarized -> 10uF
- C2: renamed from C1; value C -> 0.01uF
- J1: value Conn_01x02_Male -> (none)
- R1, R4: value R -> 1k
- R2: renamed from R3; value R -> 10k
- R3: renamed from R2; value R -> 1k
- U1: value NE555D -> (none)
Connections:
- net +9V: now also U1.4 (R)
- net pin_2: now reaches C1.1, R2.2
- net pin_2: now also U1.2 (TR), U1.6 (THR)
- net pin_3: now reaches R3.2, R4.1
- net pin_3: now also U1.3 (Q)
- net pin_7: now reaches U1.7 (DIS)
- net pin_7: now also R1.2, R2.1
