File: lab4/lab4/lab4-backups/lab4-2023-02-10_105627/lab4.kicad_sch (KiCad schematic)
At the start: 6 parts, among them J1 9 V, SW1 SW1

Commit message: Lab 6 PCB
Parts:
- C1: footprint Capacitor_THT:C_Radial_D5.0mm_H5.0mm_P2.00mm -> (none)
- D1: footprint LED_THT:LED_D5.0mm -> (none)
- J1: footprint Connector_JST:JST_PH_B2B-PH-K_1x02_P2.00mm_Vertical -> (none)
- R1: renamed from R2; footprint Resistor_THT:R_Axial_DIN0516_L15.5mm_D5.0mm_P20.32mm_Horizontal -> (none)
- R2: renamed from R1; footprint Resistor_THT:R_Axial_DIN0516_L15.5mm_D5.0mm_P20.32mm_Horizontal -> (none)
- SW1: footprint Button_Switch_THT:SW_E-Switch_EG1224_SPDT_Angled -> (none)
Changed lines of the file:
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@@
   (symbol (lib_id "Device:R") (at 110.49 69.85 180) (unit 1)
     (in_bom yes) (on_board yes) (fields_autoplaced)
-    (property "Reference" "R1" (id 0) (at 113.03 68.5799 0)
+    (property "Reference" "R2" (id 0) (at 113.03 68.5799 0)
       (effects (font (size 1.27 1.27)) (justify right))
     )
@@
       (effects (font (size 1.27 1.27)) (justify right))
     )
-    (property "Footprint" "Resistor_THT:R_Axial_DIN0516_L15.5mm_D5.0mm_P20.32mm_Horizontal" (id 2) (at 112.268 69.85 90)
+    (property "Footprint" "" (id 2) (at 112.268 69.85 90)
       (effects (font (size 1.27 1.27)) hide)
     )
@@
     (property "Reference" "SW1" (id 0) (at 90.17 54.61 0))
     (property "Value" "SW1" (id 1) (at 90.17 57.15 0))
-    (property "Footprint" "Button_Switch_THT:SW_E-Switch_EG1224_SPDT_Angled" (id 2) (at 90.17 62.23 0)
+    (property "Footprint" "" (id 2) (at 90.17 62.23 0)
       (effects (font (size 1.27 1.27)) hide)
     )
@@
       (effects (font (size 1.27 1.27)) (justify right))
     )
-    (property "Footprint" "LED_THT:LED_D5.0mm" (id 2) (at 110.49 83.82 0)
+    (property "Footprint" "" (id 2) (at 110.49 83.82 0)
       (effects (font (size 1.27 1.27)) hide)
     )
@@
       (effects (font (size 1.27 1.27)) (justify left))
     )
-    (property "Footprint" "Capacitor_THT:C_Radial_D5.0mm_H5.0mm_P2.00mm" (id 2) (at 100.0252 81.28 0)
+    (property "Footprint" "" (id 2) (at 100.0252 81.28 0)
       (effects (font (size 1.27 1.27)) hide)
     )
@@
   (symbol (lib_id "Device:R") (at 76.2 62.23 90) (unit 1)
     (in_bom yes) (on_board yes) (fields_autoplaced)
-    (property "Reference" "R2" (id 0) (at 76.2 55.88 90))
+    (property "Reference" "R1" (id 0) (at 76.2 55.88 90))
     (property "Value" "2.2 kΩ" (id 1) (at 76.2 58.42 90))
-    (property "Footprint" "Resistor_THT:R_Axial_DIN0516_L15.5mm_D5.0mm_P20.32mm_Horizontal" (id 2) (at 76.2 64.008 90)
+    (property "Footprint" "" (id 2) (at 76.2 64.008 90)
       (effects (font (size 1.27 1.27)) hide)
     )
@@
     (property "Reference" "J1" (id 0) (at 64.135 71.12 0))
     (property "Value" "9 V" (id 1) (at 64.135 73.66 0))
-    (property "Footprint" "Connector_JST:JST_PH_B2B-PH-K_1x02_P2.00mm_Vertical" (id 2) (at 63.5 76.2 0)
+    (property "Footprint" "" (id 2) (at 63.5 76.2 0)
       (effects (font (size 1.27 1.27)) hide)
     )
@@
   (symbol_instances
     (path "/c4a345d1-3bf8-404c-a2bb-b264c5df0164"
-      (reference "C1") (unit 1) (value "4.7 uF") (footprint "Capacitor_THT:C_Radial_D5.0mm_H5.0mm_P2.00mm")
+      (reference "C1") (unit 1) (value "4.7 uF") (footprint "")
     )
     (path "/afcf33ba-f6af-49e2-8fe1-c215ab12879b"
-      (reference "D1") (unit 1) (value "LED") (footprint "LED_THT:LED_D5.0mm")
+      (reference "D1") (unit 1) (value "LED") (footprint "")
     )
     (path "/fe7a6fa2-d04f-4910-bc75-9241fe904272"
-      (reference "J1") (unit 1) (value "9 V") (footprint "Connector_JST:JST_PH_B2B-PH-K_1x02_P2.00mm_Vertical")
+      (reference "J1") (unit 1) (value "9 V") (footprint "")
+    )
+    (path "/dded8343-5737-4fb2-8504-0e118044f652"
+      (reference "R1") (unit 1) (value "2.2 kΩ") (footprint "")
     )
     (path "/291efac5-afb5-4fc7-9c8b-170a0ffec518"
-      (reference "R1") (unit 1) (value "20 kΩ") (footprint "Resistor_THT:R_Axial_DIN0516_L15.5mm_D5.0mm_P20.32mm_Horizontal")
-    )
-    (path "/dded8343-5737-4fb2-8504-0e118044f652"
-      (reference "R2") (unit 1) (value "2.2 kΩ") (footprint "Resistor_THT:R_Axial_DIN0516_L15.5mm_D5.0mm_P20.32mm_Horizontal")
+      (reference "R2") (unit 1) (value "20 kΩ") (footprint "")
     )
     (path "/5ddd58a2-fb17-43f7-ba88-ec6bfbb65846"
-      (reference "SW1") (unit 1) (value "SW1") (footprint "Button_Switch_THT:SW_E-Switch_EG1224_SPDT_Angled")
+      (reference "SW1") (unit 1) (value "SW1") (footprint "")
     )
   )
