File: lab4/lab4/lab4-backups/lab4-2023-02-10_105627/lab4_Exercise2/lab4_Exercise2.kicad_sch (KiCad schematic)
At the start: 10 parts, among them J1 , U1 

Commit message: Lab 6 PCB
Parts:
- C1: footprint Capacitor_Tantalum_SMD:CP_EIA-3216-18_Kemet-A_Pad1.58x1.35mm_HandSolder -> (none)
- C2: footprint Capacitor_SMD:C_0805_2012Metric_Pad1.18x1.45mm_HandSolder -> (none)
- D1, D2: footprint LED_SMD:LED_1206_3216Metric_Pad1.42x1.75mm_HandSolder -> (none)
- J1: footprint TerminalBlock:TerminalBlock_bornier-2_P5.08mm -> (none)
- R1, R2, R3, R4: footprint Resistor_SMD:R_0805_2012Metric_Pad1.20x1.40mm_HandSolder -> (none)
- U1: footprint Package_SO:SOIC-8-1EP_3.9x4.9mm_P1.27mm_EP2.29x3mm -> Package_SO:SOIC-8_3.9x4.9mm_P1.27mm
Changed lines of the file:
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@@
       (effects (font (size 1.27 1.27)) (justify left))
     )
-    (property "Footprint" "Capacitor_SMD:C_0805_2012Metric_Pad1.18x1.45mm_HandSolder" (id 2) (at 120.3452 106.68 0)
+    (property "Footprint" "" (id 2) (at 120.3452 106.68 0)
       (effects (font (size 1.27 1.27)) hide)
     )
@@
       (effects (font (size 1.27 1.27)) (justify left))
     )
-    (property "Footprint" "Capacitor_Tantalum_SMD:CP_EIA-3216-18_Kemet-A_Pad1.58x1.35mm_HandSolder" (id 2) (at 97.4852 115.57 0)
+    (property "Footprint" "" (id 2) (at 97.4852 115.57 0)
       (effects (font (size 1.27 1.27)) hide)
     )
@@
       (effects (font (size 1.27 1.27)) (justify right))
     )
-    (property "Footprint" "LED_SMD:LED_1206_3216Metric_Pad1.42x1.75mm_HandSolder" (id 2) (at 175.26 110.49 0)
+    (property "Footprint" "" (id 2) (at 175.26 110.49 0)
       (effects (font (size 1.27 1.27)) hide)
     )
@@
       (effects (font (size 1.27 1.27)) (justify left))
     )
-    (property "Footprint" "Resistor_SMD:R_0805_2012Metric_Pad1.20x1.40mm_HandSolder" (id 2) (at 173.482 81.28 90)
+    (property "Footprint" "" (id 2) (at 173.482 81.28 90)
       (effects (font (size 1.27 1.27)) hide)
     )
@@
       (effects (font (size 1.27 1.27)) (justify left))
     )
-    (property "Footprint" "Package_SO:SOIC-8-1EP_3.9x4.9mm_P1.27mm_EP2.29x3mm" (id 2) (at 165.1 99.06 0)
+    (property "Footprint" "Package_SO:SOIC-8_3.9x4.9mm_P1.27mm" (id 2) (at 165.1 99.06 0)
       (effects (font (size 1.27 1.27)) hide)
     )
@@
       (effects (font (size 1.27 1.27)) (justify left))
     )
-    (property "Footprint" "Resistor_SMD:R_0805_2012Metric_Pad1.20x1.40mm_HandSolder" (id 2) (at 173.482 96.52 90)
+    (property "Footprint" "" (id 2) (at 173.482 96.52 90)
       (effects (font (size 1.27 1.27)) hide)
     )
@@
       (effects (font (size 1.27 1.27)) (justify right))
     )
-    (property "Footprint" "LED_SMD:LED_1206_3216Metric_Pad1.42x1.75mm_HandSolder" (id 2) (at 175.26 67.31 0)
+    (property "Footprint" "" (id 2) (at 175.26 67.31 0)
       (effects (font (size 1.27 1.27)) hide)
     )
@@
       (effects (font (size 1.27 1.27)) (justify left))
     )
-    (property "Footprint" "Resistor_SMD:R_0805_2012Metric_Pad1.20x1.40mm_HandSolder" (id 2) (at 94.742 92.71 90)
+    (property "Footprint" "" (id 2) (at 94.742 92.71 90)
       (effects (font (size 1.27 1.27)) hide)
     )
@@
       (effects (font (size 1.27 1.27)) (justify right))
     )
-    (property "Footprint" "TerminalBlock:TerminalBlock_bornier-2_P5.08mm" (id 2) (at 133.35 62.23 0)
+    (property "Footprint" "" (id 2) (at 133.35 62.23 0)
       (effects (font (size 1.27 1.27)) hide)
     )
@@
       (effects (font (size 1.27 1.27)) (justify left))
     )
-    (property "Footprint" "Resistor_SMD:R_0805_2012Metric_Pad1.20x1.40mm_HandSolder" (id 2) (at 94.742 69.85 90)
+    (property "Footprint" "" (id 2) (at 94.742 69.85 90)
       (effects (font (size 1.27 1.27)) hide)
     )
@@
     )
     (path "/3a261a9f-1698-4beb-b884-f50a0aef3d38"
-      (reference "C1") (unit 1) (value "10uF") (footprint "Capacitor_Tantalum_SMD:CP_EIA-3216-18_Kemet-A_Pad1.58x1.35mm_HandSolder")
+      (reference "C1") (unit 1) (value "10uF") (footprint "")
     )
     (path "/06849d92-0d5f-401d-a43f-98f747dab9af"
-      (reference "C2") (unit 1) (value "0.01uF") (footprint "Capacitor_SMD:C_0805_2012Metric_Pad1.18x1.45mm_HandSolder")
+      (reference "C2") (unit 1) (value "0.01uF") (footprint "")
     )
     (path "/76d6cc1a-cf83-41f9-804e-d548a442661c"
-      (reference "D1") (unit 1) (value "LED") (footprint "LED_SMD:LED_1206_3216Metric_Pad1.42x1.75mm_HandSolder")
+      (reference "D1") (unit 1) (value "LED") (footprint "")
     )
     (path "/5010e7c3-2ea5-482f-9fa9-86683560bd9e"
-      (reference "D2") (unit 1) (value "LED") (footprint "LED_SMD:LED_1206_3216Metric_Pad1.42x1.75mm_HandSolder")
+      (reference "D2") (unit 1) (value "LED") (footprint "")
     )
     (path "/cd4a55ee-2a2c-4e20-8755-348ec09b906e"
-      (reference "J1") (unit 1) (value " ") (footprint "TerminalBlock:TerminalBlock_bornier-2_P5.08mm")
+      (reference "J1") (unit 1) (value " ") (footprint "")
     )
     (path "/fe38d667-9b7c-498a-8e7f-0229027aac54"
-      (reference "R1") (unit 1) (value "1k") (footprint "Resistor_SMD:R_0805_2012Metric_Pad1.20x1.40mm_HandSolder")
+      (reference "R1") (unit 1) (value "1k") (footprint "")
     )
     (path "/7d7d7875-4d57-43ba-9372-599bca77c45a"
-      (reference "R2") (unit 1) (value "10k") (footprint "Resistor_SMD:R_0805_2012Metric_Pad1.20x1.40mm_HandSolder")
+      (reference "R2") (unit 1) (value "10k") (footprint "")
     )
     (path "/588701a5-c2b5-4037-a1d4-5f9984b05d36"
-      (reference "R3") (unit 1) (value "1k") (footprint "Resistor_SMD:R_0805_2012Metric_Pad1.20x1.40mm_HandSolder")
+      (reference "R3") (unit 1) (value "1k") (footprint "")
     )
     (path "/63cc3412-2105-4250-b06a-5152d4882c6b"
-      (reference "R4") (unit 1) (value "1k") (footprint "Resistor_SMD:R_0805_2012Metric_Pad1.20x1.40mm_HandSolder")
+      (reference "R4") (unit 1) (value "1k") (footprint "")
     )
     (path "/61a7e486-8865-4599-b7c7-64a51809fdc6"
-      (reference "U1") (unit 1) (value " ") (footprint "Package_SO:SOIC-8-1EP_3.9x4.9mm_P1.27mm_EP2.29x3mm")
-    )
-  )
+      (reference "U1") (unit 1) (value " ") (footprint "Package_SO:SOIC-8_3.9x4.9mm_P1.27mm")
+    )
+  )
